File: discipline-pcb.kicad_pcb (KiCad board)
At the start: 2 copper layers, 304.9 x 122.8 mm, 180 parts, among them J1 AVR-ISP-6, SW1 KEYSW, SW10 KEYSW, SW11 KEYSW, SW12 KEYSW, SW13 KEYSW, SW14 KEYSW, SW15 KEYSW, SW16 KEYSW, SW17 KEYSW, SW18 KEYSW, SW19 KEYSW, SW2 KEYSW, SW20 KEYSW, SW21 KEYSW, SW22 KEYSW, SW23 KEYSW, SW24 KEYSW, SW25 KEYSW, SW26 KEYSW, SW27 KEYSW, SW28 KEYSW, SW29 KEYSW, SW3 KEYSW, SW30 KEYSW, SW31 KEYSW, SW32 KEYSW, SW33 KEYSW, SW34 KEYSW, SW35 KEYSW, SW36 KEYSW, SW37 KEYSW, SW38 KEYSW, SW39 KEYSW, SW4 KEYSW, SW40 KEYSW, SW41 KEYSW, SW42 KEYSW, SW43 KEYSW, SW44 KEYSW, SW45 KEYSW, SW46 KEYSW, SW47 KEYSW, SW48 KEYSW, SW49 KEYSW, SW5 KEYSW, SW50 KEYSW, SW51 KEYSW, SW52 KEYSW, SW53 KEYSW, SW54 KEYSW, SW55 KEYSW, SW56 KEYSW, SW57 KEYSW, SW58 KEYSW, SW59 KEYSW, SW6 KEYSW, SW60 KEYSW, SW61 KEYSW, SW62 KEYSW, SW63 KEYSW, SW64 KEYSW, SW65 KEYSW, SW66 KEYSW, SW67 KEYSW, SW68 KEYSW, SW69 KEYSW, SW7 KEYSW, SW70 KEYSW, SW71 KEYSW, SW72 KEYSW, SW73 KEYSW, SW74 KEYSW, SW8 KEYSW, SW9 KEYSW, U1 ATmega32A-PU, Y1 Crystal

Commit message: Revert "Update discipline-pcb.kicad_pcb"
This reverts commit 5b5a9406b507a9cf9a6000bfc02bb23341a56901.
Parts:
- removed the G*** at (161.9, 158.9)
- removed SW69: KEYSW, cftkb:SW_Cherry_MX1A_1.25u_PCBNOSCREEN
- removed SW70, SW71, SW73, SW74: KEYSW, cftkb:SW_Cherry_MX1A_1.50u_PCBNOSCREEN
- removed SW72: KEYSW, Button_Switch_Keyboard:SW_Cherry_MX1A_1.00u_PCB-NOSCREEN
- added G***: LOGO, logos:DISCIPLINE_SMALL_COPPER, F.Cu at (161.9, 158.9)
- added SW31: KEYSW, Button_Switch_Keyboard:SW_Cherry_MX1A_1.25u_PCBNOSCREEN, F.Cu at (75.0, 123.0)
- added SW59: KEYSW, Button_Switch_Keyboard:SW_Cherry_MX1A_1.50u_PCBNOSCREEN, F.Cu at (77.4, 161.1)
- added SW61: KEYSW, Button_Switch_Keyboard:SW_Cherry_MX1A_1.50u_PCBNOSCREEN, F.Cu at (106.0, 161.1)
- added SW62: KEYSW, Button_Switch_Keyboard:SW_Cherry_MX1A_1.00u_PCB-NOSCREEN, F.Cu at (187.0, 161.1)
- added SW63: KEYSW, Button_Switch_Keyboard:SW_Cherry_MX1A_1.50u_PCBNOSCREEN, F.Cu at (268.0, 161.1)
- added SW64: KEYSW, Button_Switch_Keyboard:SW_Cherry_MX1A_1.50u_PCBNOSCREEN, F.Cu at (296.5, 161.1)
- BOOT1, RESET1: footprint cftkb:SW_PUSH_6mm -> Button_Switch_THT:SW_PUSH_6mm
- C1, C2: footprint cftkb:C_Disc_D3.0mm_W1.6mm_P2.50mm -> Capacitor_THT:C_Disc_D3.0mm_W1.6mm_P2.50mm
- C3: footprint cftkb:CP_Radial_D4.0mm_P1.50mm -> Capacitor_THT:CP_Radial_D4.0mm_P1.50mm
- C4, C5: footprint cftkb:C_Disc_D4.3mm_W1.9mm_P5.00mm -> Capacitor_THT:C_Disc_D4.3mm_W1.9mm_P5.00mm
- D1, D10, D11, D12, D13, D14, D15, D16, D17, D18, D19, D2, D20, D21, D22, D23, D24, D25, D26, D27, D28, D29, D3, D30, D31, D32, D33, D34, D35, D36, D37, D38, D39, D4, D40, D41, D42, D43, D44, D45, D46, D47, D48, D49, D5, D50, D51, D52, D53, D54, D55, D56, D57, D58, D59, D6, D60, D61, D62, D63, D64, D65, D66, D67, D68, D7, D8, D9: footprint cftkb:D_DO-35_SOD27_P5.08mm_Horizontal -> Diode_THT:D_DO-35_SOD27_P5.08mm_Horizontal
- D69, D70: value 3.6V -> 3V6; footprint cftkb:D_DO-35_SOD27_P5.08mm_Horizontal -> Diode_THT:D_DO-35_SOD27_P5.08mm_Horizontal
- F1: footprint cftkb:polyfuse_5.1mm -> keyboard_parts:polyfuse_5.1mm
- J1: footprint cftkb:AVR_ICSP_3x2 -> keyboard_parts:AVR_ICSP_3x2
- LED1: footprint cftkb:LED_D3.0mm -> LED_THT:LED_D3.0mm
- R1, R2, R3, R4, R6: footprint cftkb:R_Axial_DIN0204_L3.6mm_D1.6mm_P7.62mm_Horizontal -> Resistor_THT:R_Axial_DIN0204_L3.6mm_D1.6mm_P7.62mm_Horizontal
- R5: value 1.5k -> 1.5K; footprint cftkb:R_Axial_DIN0204_L3.6mm_D1.6mm_P7.62mm_Horizontal -> Resistor_THT:R_Axial_DIN0204_L3.6mm_D1.6mm_P7.62mm_Horizontal
- R7: value 10k -> 10K; footprint cftkb:R_Axial_DIN0204_L3.6mm_D1.6mm_P7.62mm_Horizontal -> Resistor_THT:R_Axial_DIN0204_L3.6mm_D1.6mm_P7.62mm_Horizontal
- ST62: footprint cftkb:MX-6.25U-Stabilizer -> MX_Alps_Hybrid:MX-6.25U-Stabilizer; moved to B.Cu
- ST62: renamed from ST72; footprint cftkb:MX-7U-Stabilizer -> MX_Alps_Hybrid:MX-7U-Stabilizer
- SW1, SW10, SW11, SW12, SW13, SW15, SW17, SW18, SW19, SW2, SW20, SW21, SW22, SW23, SW24, SW25, SW26, SW27, SW28, SW3, SW30, SW32, SW33, SW34, SW35, SW36, SW37, SW38, SW39, SW4, SW40, SW41, SW42, SW44, SW46, SW47, SW48, SW49, SW5, SW50, SW51, SW52, SW53, SW54, SW55, SW57, SW58, SW6, SW62, SW63, SW64, SW65, SW66, SW67, SW68, SW7, SW8, SW9: footprint cftkb:SW_Cherry_MX1A_1.00u_PCB-NOSCREEN -> Button_Switch_Keyboard:SW_Cherry_MX1A_1.00u_PCB-NOSCREEN
- SW14: footprint cftkb:SW_Cherry_MX1A_2.00u_PCBNOSCREEN -> Button_Switch_Keyboard:SW_Cherry_MX1A_2.00u_PCBNOSCREEN
- SW16, SW29: footprint cftkb:SW_Cherry_MX1A_1.50u_PCBNOSCREEN -> Button_Switch_Keyboard:SW_Cherry_MX1A_1.50u_PCBNOSCREEN
- SW31, SW56: footprint cftkb:SW_Cherry_MX1A_1.75u_PCBNOSCREEN -> Button_Switch_Keyboard:SW_Cherry_MX1A_1.75u_PCBNOSCREEN
- SW43, SW45: footprint cftkb:SW_Cherry_MX1A_2.25u_PCBNOSCREEN -> Button_Switch_Keyboard:SW_Cherry_MX1A_2.25u_PCBNOSCREEN
- SW59, SW60, SW61: footprint cftkb:SW_Cherry_MX1A_1.25u_PCBNOSCREEN -> Button_Switch_Keyboard:SW_Cherry_MX1A_1.25u_PCBNOSCREEN
- USB1: value USB_C_GCT_USB4085 -> USB_C_USB4085; footprint cftkb:USB_C_GCT_USB4085 -> Type-C:USB_C_GCT_USB4085
- Y1: footprint cftkb:Crystal_HC49-4H_Vertical -> Crystal:Crystal_HC49-4H_Vertical
- turned ST62 to 180 degrees
Connections:
- net Net-(U1-Pad15) renamed boot_led

Commit message: Update discipline-pcb.kicad_pcb
Parts:
- removed the G*** at (161.9, 158.9)
- removed the SW31 at (75.0, 123.0)
- removed the SW59 at (77.4, 161.1)
- removed the SW61 at (106.0, 161.1)
- removed the SW62 at (187.0, 161.1)
- removed the SW63 at (268.0, 161.1)
- removed the SW64 at (296.5, 161.1)
- added G***: LOGO, cftkb:DISCIPLINE_SMALL_COPPER, F.Cu at (161.9, 158.9)
- added SW69: KEYSW, cftkb:SW_Cherry_MX1A_1.25u_PCBNOSCREEN, F.Cu at (75.1, 123.1)
- added SW70: KEYSW, cftkb:SW_Cherry_MX1A_1.50u_PCBNOSCREEN, F.Cu at (77.5, 161.2)
- added SW71: KEYSW, cftkb:SW_Cherry_MX1A_1.50u_PCBNOSCREEN, F.Cu at (106.0, 161.2)
- added SW72: KEYSW, Button_Switch_Keyboard:SW_Cherry_MX1A_1.00u_PCB-NOSCREEN, F.Cu at (187.0, 161.1)
- added SW73: KEYSW, cftkb:SW_Cherry_MX1A_1.50u_PCBNOSCREEN, F.Cu at (268.0, 161.2)
- added SW74: KEYSW, cftkb:SW_Cherry_MX1A_1.50u_PCBNOSCREEN, F.Cu at (296.5, 161.2)
- BOOT1, RESET1: footprint Button_Switch_THT:SW_PUSH_6mm -> cftkb:SW_PUSH_6mm
- C1, C2: footprint Capacitor_THT:C_Disc_D3.0mm_W1.6mm_P2.50mm -> cftkb:C_Disc_D3.0mm_W1.6mm_P2.50mm
- C3: footprint Capacitor_THT:CP_Radial_D4.0mm_P1.50mm -> cftkb:CP_Radial_D4.0mm_P1.50mm
- C4, C5: footprint Capacitor_THT:C_Disc_D4.3mm_W1.9mm_P5.00mm -> cftkb:C_Disc_D4.3mm_W1.9mm_P5.00mm
- D1, D10, D11, D12, D13, D14, D15, D16, D17, D18, D19, D2, D20, D21, D22, D23, D24, D25, D26, D27, D28, D29, D3, D30, D31, D32, D33, D34, D35, D36, D37, D38, D39, D4, D40, D41, D42, D43, D44, D45, D46, D47, D48, D49, D5, D50, D51, D52, D53, D54, D55, D56, D57, D58, D59, D6, D60, D61, D62, D63, D64, D65, D66, D67, D68, D7, D8, D9: footprint Diode_THT:D_DO-35_SOD27_P5.08mm_Horizontal -> cftkb:D_DO-35_SOD27_P5.08mm_Horizontal
- D69, D70: value 3V6 -> 3.6V; footprint Diode_THT:D_DO-35_SOD27_P5.08mm_Horizontal -> cftkb:D_DO-35_SOD27_P5.08mm_Horizontal
- F1: footprint keyboard_parts:polyfuse_5.1mm -> cftkb:polyfuse_5.1mm
- J1: footprint keyboard_parts:AVR_ICSP_3x2 -> cftkb:AVR_ICSP_3x2
- LED1: footprint LED_THT:LED_D3.0mm -> cftkb:LED_D3.0mm
- R1, R2, R3, R4, R6: footprint Resistor_THT:R_Axial_DIN0204_L3.6mm_D1.6mm_P7.62mm_Horizontal -> cftkb:R_Axial_DIN0204_L3.6mm_D1.6mm_P7.62mm_Horizontal
- R5: value 1.5K -> 1.5k; footprint Resistor_THT:R_Axial_DIN0204_L3.6mm_D1.6mm_P7.62mm_Horizontal -> cftkb:R_Axial_DIN0204_L3.6mm_D1.6mm_P7.62mm_Horizontal
- R7: value 10K -> 10k; footprint Resistor_THT:R_Axial_DIN0204_L3.6mm_D1.6mm_P7.62mm_Horizontal -> cftkb:R_Axial_DIN0204_L3.6mm_D1.6mm_P7.62mm_Horizontal
- ST62: footprint MX_Alps_Hybrid:MX-6.25U-Stabilizer -> cftkb:MX-6.25U-Stabilizer; moved to F.Cu
- ST72: renamed from ST62; footprint MX_Alps_Hybrid:MX-7U-Stabilizer -> cftkb:MX-7U-Stabilizer
- SW1, SW10, SW11, SW12, SW13, SW15, SW17, SW18, SW19, SW2, SW20, SW21, SW22, SW23, SW24, SW25, SW26, SW27, SW28, SW3, SW30, SW32, SW33, SW34, SW35, SW36, SW37, SW38, SW39, SW4, SW40, SW41, SW42, SW44, SW46, SW47, SW48, SW49, SW5, SW50, SW51, SW52, SW53, SW54, SW55, SW57, SW58, SW6, SW62, SW63, SW64, SW65, SW66, SW67, SW68, SW7, SW8, SW9: footprint Button_Switch_Keyboard:SW_Cherry_MX1A_1.00u_PCB-NOSCREEN -> cftkb:SW_Cherry_MX1A_1.00u_PCB-NOSCREEN
- SW14: footprint Button_Switch_Keyboard:SW_Cherry_MX1A_2.00u_PCBNOSCREEN -> cftkb:SW_Cherry_MX1A_2.00u_PCBNOSCREEN
- SW16, SW29: footprint Button_Switch_Keyboard:SW_Cherry_MX1A_1.50u_PCBNOSCREEN -> cftkb:SW_Cherry_MX1A_1.50u_PCBNOSCREEN
- SW31, SW56: footprint Button_Switch_Keyboard:SW_Cherry_MX1A_1.75u_PCBNOSCREEN -> cftkb:SW_Cherry_MX1A_1.75u_PCBNOSCREEN
- SW43, SW45: footprint Button_Switch_Keyboard:SW_Cherry_MX1A_2.25u_PCBNOSCREEN -> cftkb:SW_Cherry_MX1A_2.25u_PCBNOSCREEN
- SW59, SW60, SW61: footprint Button_Switch_Keyboard:SW_Cherry_MX1A_1.25u_PCBNOSCREEN -> cftkb:SW_Cherry_MX1A_1.25u_PCBNOSCREEN
- USB1: value USB_C_USB4085 -> USB_C_GCT_USB4085; footprint Type-C:USB_C_GCT_USB4085 -> cftkb:USB_C_GCT_USB4085
- Y1: footprint Crystal:Crystal_HC49-4H_Vertical -> cftkb:Crystal_HC49-4H_Vertical
- turned ST62 to 0 degrees
Connections:
- net boot_led renamed Net-(U1-Pad15)
