File: discipline-pcb.kicad_pcb (KiCad board)
At the start: 2 copper layers, 304.9 x 122.8 mm, 180 parts, among them J1 AVR-ISP-6, SW1 KEYSW, SW10 KEYSW, SW11 KEYSW, SW12 KEYSW, SW13 KEYSW, SW14 KEYSW, SW15 KEYSW, SW16 KEYSW, SW17 KEYSW, SW18 KEYSW, SW19 KEYSW, SW2 KEYSW, SW20 KEYSW, SW21 KEYSW, SW22 KEYSW, SW23 KEYSW, SW24 KEYSW, SW25 KEYSW, SW26 KEYSW, SW27 KEYSW, SW28 KEYSW, SW29 KEYSW, SW3 KEYSW, SW30 KEYSW, SW31 KEYSW, SW32 KEYSW, SW33 KEYSW, SW34 KEYSW, SW35 KEYSW, SW36 KEYSW, SW37 KEYSW, SW38 KEYSW, SW39 KEYSW, SW4 KEYSW, SW40 KEYSW, SW41 KEYSW, SW42 KEYSW, SW43 KEYSW, SW44 KEYSW, SW45 KEYSW, SW46 KEYSW, SW47 KEYSW, SW48 KEYSW, SW49 KEYSW, SW5 KEYSW, SW50 KEYSW, SW51 KEYSW, SW52 KEYSW, SW53 KEYSW, SW54 KEYSW, SW55 KEYSW, SW56 KEYSW, SW57 KEYSW, SW58 KEYSW, SW59 KEYSW, SW6 KEYSW, SW60 KEYSW, SW61 KEYSW, SW62 KEYSW, SW63 KEYSW, SW64 KEYSW, SW65 KEYSW, SW66 KEYSW, SW67 KEYSW, SW68 KEYSW, SW69 KEYSW, SW7 KEYSW, SW70 KEYSW, SW71 KEYSW, SW72 KEYSW, SW73 KEYSW, SW74 KEYSW, SW8 KEYSW, SW9 KEYSW, U1 ATmega32A-PU, Y1 Crystal

Commit message: Update discipline-pcb.kicad_pcb
Parts:
- moved REF** 8.28 mm to (315.9, 161.1)
- moved SW54 8.28 mm to (261.1, 146.8)
- moved SW56 8.28 mm to (306.4, 146.8)
- moved SW64 8.28 mm to (275.5, 165.9)
- moved SW65 8.28 mm to (313.5, 165.9)
- moved SW68 8.28 mm to (294.5, 165.9)
- moved C2 8.28 mm to (327.7, 82.0)
- moved C3 8.28 mm to (284.5, 70.4)
- moved D15 8.28 mm to (275.5, 71.2)
- moved D39 8.28 mm to (171.4, 69.5)
- moved D40 8.28 mm to (184.0, 69.5)
- moved D59 8.28 mm to (259.8, 69.5)
- moved D63 8.28 mm to (250.3, 71.2)
- moved D67 8.28 mm to (262.9, 71.2)
- moved D69 8.28 mm to (286.2, 71.9)
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
Commit message: Update to V2, add ISO support, update license
Parts:
- added D71: , cftkb:D_DO-35_SOD27_P5.08mm_Horizontal, F.Cu at (96.7, 147.0)
- added G***: LOGO, logos:rev1-1_16mm_copper, B.Cu at (155.2, 174.0)
- added G***: LOGO, logos:coseyfannitutti_16mm, F.Cu at (155.1, 168.3)
- added G***: LOGO, logos:rev1-1_16mm_mask, B.Cu at (155.2, 174.0)
- added G***: LOGO, logos:coseyfannitutti_rev1_16mm_copper, B.Cu at (155.3, 168.3)
- added G***: LOGO, logos:coseyfannitutti_16mm, B.Cu at (155.3, 168.3)
- added G***: LOGO, logos:DISCIPLINE_SMALL_COPPER, B.Cu at (155.2, 163.6)
- added G***: LOGO, logos:DISCIPLINE_SMALL_MASK, B.Cu at (155.2, 163.6)
- added G***: LOGO, logos:rev1-1_16mm_copper, F.Cu at (155.1, 174.0)
- added G***: LOGO, logos:rev1-1_16mm_mask, F.Cu at (155.1, 174.0)
- added G***: LOGO, logos:coseyfannitutti_rev1_16mm_copper, F.Cu at (155.1, 168.3)
- added REF**: MountingHole_2.2mm_M2_Pad, MountingHole:MountingHole_2.2mm_M2_Pad, F.Cu at (206.2, 61.7)
- added REF**: MountingHole_2.2mm_M2_Pad, MountingHole:MountingHole_2.2mm_M2_Pad, F.Cu at (206.2, 80.4)
- added SW75: KEYSW, cftkb:SW_Cherry_MX1A_1.00u_PCB-NOSCREEN, F.Cu at (89.7, 146.8)
- added SW76: KEYSW, cftkb:SW_Cherry_MX1A_ISOEnter_PCB_ReversedStabilizer, F.Cu at (330.2, 118.3)
- added SW77: KEYSW, cftkb:SW_Cherry_MX1A_1.00u_PCB-NOSCREEN, F.Cu at (308.8, 127.8)
- added SW78: KEYSW, cftkb:SW_Cherry_MX1A_1.25u_PCBNOSCREEN, F.Cu at (68.3, 146.8)
- R1, R2, R3, R4, R5, R6, R7: footprint cftkb:R_Axial_DIN0204_L3.6mm_D1.6mm_P7.62mm_Horizontal -> cftkb:R_Axial_DIN0204_L3.6mm_D1.6mm_P5.08mm_Horizontal
- SW63, SW64: footprint cftkb:SW_Cherry_MX1A_1.00u_PCB-NOSCREEN -> cftkb:SW_Cherry_MX1A_1.25u_PCBNOSCREEN
- moved R1 1.27 mm to (290.0, 70.6)
- moved R2 1.27 mm to (290.0, 68.1)
- moved R3 1.27 mm to (295.1, 73.2)
- moved R4 1.27 mm to (295.1, 75.6)
- moved R5 1.27 mm to (295.1, 78.1)
- moved R6 1.27 mm to (290.0, 65.6)
- moved R7 1.27 mm to (295.1, 63.1)
- moved REF** 0.72 mm to (57.8, 80.4)
- moved REF** 0.72 mm to (354.7, 80.4)
- moved REF** 0.72 mm to (57.8, 61.7)
- moved REF** 0.72 mm to (354.7, 61.7)
Routing:
- net row3: track 287.2 -> 404.8 mm, vias 3 -> 7
- net GND: track 241.1 -> 223.5 mm, vias 36 -> 48
- net Net-(D71-Pad2): track 0.00 -> 15.0 mm
- net col13: track 146.9 -> 161.3 mm
- net Net-(D43-Pad2): track 140.6 -> 153.6 mm
- net Net-(D29-Pad2): track 117.7 -> 127.9 mm
- net col0: track 355.0 -> 364.4 mm, vias 0 -> 2
- net Net-(D45-Pad2): track 76.5 -> 85.1 mm
- net row1: track 268.1 -> 272.6 mm, vias 2 -> 4
- net row0: track 263.1 -> 267.2 mm
- net row4: track 296.4 -> 299.4 mm
- net D+: track 42.4 -> 45.3 mm
- net +5V: track 147.9 -> 145.4 mm
- net col2: track 329.2 -> 331.4 mm, vias 0 -> 2
- net col4: track 259.3 -> 261.3 mm, vias 0 -> 2
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Other:
- board text added: "1.1"
- board text added: "1.25U ISO"
- board text added: "1U ISO"
- board text added: "2.25U ANSI"
- board text added: "7/2/2019 - updated 12/3/2019"
- board text added: "ANSI ENTER"
- board text added: "DISCIPLINE - 65% keyboard assembled with only through hole components"
- board text added: "ISO"
- board text added: "ISO ENTER"
- board text removed: "1"
- board text removed: "7/2/2019"
- board text removed: "DISCIPLINE - 65% keyboard made with only through hole components"
- board text removed: "coseyfannitutti 2019 rev1"

Commit message: Fix broken ref Y1 on pcb
Connections:
- BOOT1 pad 1: GND -> boot
- BOOT1 pad 2: boot -> GND
- RESET1 pad 1: GND -> reset
- RESET1 pad 2: reset -> GND
