File: discipline-pcb.sch (KiCad schematic (older format))
At the start: 158 parts, among them J1 AVR-ISP-6, SW1 KEYSW, SW10 KEYSW, SW11 KEYSW, SW12 KEYSW, SW13 KEYSW, SW14 KEYSW, SW15 KEYSW, SW16 KEYSW, SW17 KEYSW, SW18 KEYSW, SW19 KEYSW, SW2 KEYSW, SW20 KEYSW, SW21 KEYSW, SW22 KEYSW, SW23 KEYSW, SW24 KEYSW, SW25 KEYSW, SW26 KEYSW, SW27 KEYSW, SW28 KEYSW, SW29 KEYSW, SW3 KEYSW, SW30 KEYSW, SW31 KEYSW, SW32 KEYSW, SW33 KEYSW, SW34 KEYSW, SW35 KEYSW, SW36 KEYSW, SW37 KEYSW, SW38 KEYSW, SW39 KEYSW, SW4 KEYSW, SW40 KEYSW, SW41 KEYSW, SW42 KEYSW, SW43 KEYSW, SW44 KEYSW, SW45 KEYSW, SW46 KEYSW, SW47 KEYSW, SW48 KEYSW, SW49 KEYSW, SW5 KEYSW, SW50 KEYSW, SW51 KEYSW, SW52 KEYSW, SW53 KEYSW, SW54 KEYSW, SW55 KEYSW, SW56 KEYSW, SW57 KEYSW, SW58 KEYSW, SW59 KEYSW, SW6 KEYSW, SW60 KEYSW, SW61 KEYSW, SW62 KEYSW, SW63 KEYSW, SW64 KEYSW, SW65 KEYSW, SW66 KEYSW, SW67 KEYSW, SW68 KEYSW, SW7 KEYSW, SW8 KEYSW, SW9 KEYSW, U1 ATmega32A-PU, Y1 Crystal

Commit message: Update discipline-pcb.sch
Parts:
- U1: symbol MCU_Microchip_ATmega:ATmega32A-PU -> discipline-pcb-rescue:ATmega32A-PU-MCU_Microchip_ATmega
Changed lines of the file:
@@
 EESchema Schematic File Version 4
 LIBS:discipline-pcb-cache
-EELAYER 26 0
+EELAYER 30 0
 EELAYER END
 $Descr A3 16535 11693
@@
 reset
 $Comp
-L MCU_Microchip_ATmega:ATmega32A-PU U1
+L discipline-pcb-rescue:ATmega32A-PU-MCU_Microchip_ATmega U1
 U 1 1 5D1828C7
 P 4000 8250
@@
 Wire Wire Line
 	13350 2900 13350 5250
-$Comp
-L keyboard_parts:GND #PWR?
-U 1 1 5D3CA2AB
-P 5550 10300
-F 0 "#PWR?" H 5550 10350 20  0001 C CNN
-F 1 "GND" H 5550 10200 30  0000 C CNN
-F 2 "" H 5550 10300 60  0000 C CNN
-F 3 "" H 5550 10300 60  0000 C CNN
-	1    5550 10300
-	1    0    0    -1
-$EndComp
 NoConn ~ 3400 7150
 NoConn ~ 4600 7050
@@
 NoConn ~ 4600 9250
 NoConn ~ 4600 9350
+$Comp
+L power:GND #PWR?
+U 1 1 5DA49277
+P 5550 10300
+F 0 "#PWR?" H 5550 10050 50  0001 C CNN
+F 1 "GND" H 5555 10127 50  0000 C CNN
+F 2 "" H 5550 10300 50  0001 C CNN
+F 3 "" H 5550 10300 50  0001 C CNN
+	1    5550 10300
+	1    0    0    -1
+$EndComp
 $EndSCHEMATC

Commit message: add schematic symbols for alternate switches so netlist updates properly
Parts:
- added SW69: KEYSW, cftkb:SW_Cherry_MX1A_1.25u_PCBNOSCREEN, symbol keyboard_parts:KEYSW
- added SW70, SW71, SW73, SW74: KEYSW, cftkb:SW_Cherry_MX1A_1.50u_PCBNOSCREEN, symbol keyboard_parts:KEYSW
- added SW72: KEYSW, cftkb:SW_Cherry_MX1A_1.00u_PCB-NOSCREEN, symbol keyboard_parts:KEYSW
- BOOT1, RESET1: footprint Button_Switch_THT:SW_PUSH_6mm -> cftkb:SW_PUSH_6mm
- C1, C2: footprint Capacitor_THT:C_Disc_D3.0mm_W1.6mm_P2.50mm -> cftkb:D_DO-35_SOD27_P5.08mm_Horizontal
- C3: footprint Capacitor_THT:CP_Radial_D4.0mm_P1.50mm -> cftkb:D_DO-35_SOD27_P5.08mm_Horizontal
- C4, C5: footprint Capacitor_THT:C_Disc_D4.3mm_W1.9mm_P5.00mm -> cftkb:D_DO-35_SOD27_P5.08mm_Horizontal
- D1, D10, D11, D12, D13, D14, D15, D16, D17, D18, D19, D2, D20, D21, D22, D23, D24, D25, D26, D27, D28, D29, D3, D30, D31, D32, D33, D34, D35, D36, D37, D38, D39, D4, D40, D41, D42, D43, D44, D45, D46, D47, D48, D49, D5, D50, D51, D52, D53, D54, D55, D56, D57, D58, D59, D6, D60, D61, D62, D63, D64, D65, D66, D67, D68, D69, D7, D70, D8, D9: footprint Diode_THT:D_DO-35_SOD27_P5.08mm_Horizontal -> cftkb:D_DO-35_SOD27_P5.08mm_Horizontal
- F1: footprint keyboard_parts:polyfuse_5.1mm -> cftkb:polyfuse_5.1mm
- J1: footprint (none) -> cftkb:AVR_ICSP_3x2
- LED1: footprint LED_THT:LED_D3.0mm -> cftkb:LED_D3.0mm
- R1, R2, R3, R4, R5, R6, R7: footprint Resistor_THT:R_Axial_DIN0204_L3.6mm_D1.6mm_P7.62mm_Horizontal -> cftkb:R_Axial_DIN0204_L3.6mm_D1.6mm_P7.62mm_Horizontal
- SW1, SW10, SW11, SW12, SW13, SW15, SW17, SW18, SW19, SW2, SW20, SW21, SW22, SW23, SW24, SW25, SW26, SW27, SW28, SW3, SW30, SW32, SW33, SW34, SW35, SW36, SW37, SW38, SW39, SW4, SW40, SW41, SW42, SW44, SW46, SW47, SW48, SW49, SW5, SW50, SW51, SW52, SW53, SW54, SW55, SW57, SW58, SW6, SW62, SW65, SW66, SW67, SW68, SW7, SW8, SW9: footprint Button_Switch_Keyboard:SW_Cherry_MX1A_1.00u_PCB-NOSCREEN -> cftkb:SW_Cherry_MX1A_1.00u_PCB-NOSCREEN
- SW14: footprint Button_Switch_Keyboard:SW_Cherry_MX1A_2.00u_PCBNOSCREEN -> cftkb:SW_Cherry_MX1A_2.00u_PCBNOSCREEN
- SW16, SW29: footprint Button_Switch_Keyboard:SW_Cherry_MX1A_1.50u_PCBNOSCREEN -> cftkb:SW_Cherry_MX1A_1.50u_PCBNOSCREEN
- SW31, SW56: footprint Button_Switch_Keyboard:SW_Cherry_MX1A_1.75u_PCBNOSCREEN -> cftkb:SW_Cherry_MX1A_1.75u_PCBNOSCREEN
- SW43, SW45: footprint Button_Switch_Keyboard:SW_Cherry_MX1A_2.25u_PCBNOSCREEN -> cftkb:SW_Cherry_MX1A_2.25u_PCBNOSCREEN
- SW59, SW60, SW61, SW63, SW64: footprint Button_Switch_Keyboard:SW_Cherry_MX1A_1.25u_PCBNOSCREEN -> cftkb:SW_Cherry_MX1A_1.25u_PCBNOSCREEN
- U1: footprint Package_DIP:DIP-40_W15.24mm -> cftkb:DIP-40_W15.24mm
- USB1: footprint Type-C:USB_C_GCT_USB4085 -> cftkb:USB_C_GCT_USB4085
- Y1: footprint Crystal:Crystal_HC49-4H_Vertical -> cftkb:Crystal_HC49-4H_Vertical
Connections:
- wire segments 271 -> 342
