File: discipline-pcb.sch (KiCad schematic (older format))
At the start: 158 parts, among them J1 AVR-ISP-6, SW1 KEYSW, SW10 KEYSW, SW11 KEYSW, SW12 KEYSW, SW13 KEYSW, SW14 KEYSW, SW15 KEYSW, SW16 KEYSW, SW17 KEYSW, SW18 KEYSW, SW19 KEYSW, SW2 KEYSW, SW20 KEYSW, SW21 KEYSW, SW22 KEYSW, SW23 KEYSW, SW24 KEYSW, SW25 KEYSW, SW26 KEYSW, SW27 KEYSW, SW28 KEYSW, SW29 KEYSW, SW3 KEYSW, SW30 KEYSW, SW31 KEYSW, SW32 KEYSW, SW33 KEYSW, SW34 KEYSW, SW35 KEYSW, SW36 KEYSW, SW37 KEYSW, SW38 KEYSW, SW39 KEYSW, SW4 KEYSW, SW40 KEYSW, SW41 KEYSW, SW42 KEYSW, SW43 KEYSW, SW44 KEYSW, SW45 KEYSW, SW46 KEYSW, SW47 KEYSW, SW48 KEYSW, SW49 KEYSW, SW5 KEYSW, SW50 KEYSW, SW51 KEYSW, SW52 KEYSW, SW53 KEYSW, SW54 KEYSW, SW55 KEYSW, SW56 KEYSW, SW57 KEYSW, SW58 KEYSW, SW59 KEYSW, SW6 KEYSW, SW60 KEYSW, SW61 KEYSW, SW62 KEYSW, SW63 KEYSW, SW64 KEYSW, SW65 KEYSW, SW66 KEYSW, SW67 KEYSW, SW68 KEYSW, SW7 KEYSW, SW8 KEYSW, SW9 KEYSW, U1 ATmega32A-PU, Y1 Crystal

Commit message: clean up symbol labels
Parts:
- R3, R4: value 68R -> 75R
Changed lines of the file:
@@
 P 8550 7050
 F 0 "R3" V 8450 7050 50  0000 C CNN
-F 1 "68R" V 8550 7050 50  0000 C CNN
+F 1 "75R" V 8550 7050 39  0000 C CNN
 F 2 "Resistor_THT:R_Axial_DIN0204_L3.6mm_D1.6mm_P7.62mm_Horizontal" H 8550 7050 50  0001 C CNN
 F 3 "~" H 8550 7050 50  0001 C CNN
@@
 P 8550 7150
 F 0 "R4" V 8650 7150 50  0000 C CNN
-F 1 "68R" V 8550 7150 50  0000 C CNN
+F 1 "75R" V 8550 7150 39  0000 C CNN
 F 2 "Resistor_THT:R_Axial_DIN0204_L3.6mm_D1.6mm_P7.62mm_Horizontal" H 8550 7150 50  0001 C CNN
 F 3 "~" H 8550 7150 50  0001 C CNN

Commit message: change fuse value
change fuse value from 100mA to 500mA. 100mA is fine for this use, but 500mA is USB 2.0 standard
Parts:
- F1: value 100mA -> 500mA
Changed lines of the file:
@@
 P 7800 6300
 F 0 "F1" H 7868 6346 50  0000 L CNN
-F 1 "100mA" H 7868 6255 50  0000 L CNN
+F 1 "500mA" H 7868 6255 50  0000 L CNN
 F 2 "keyboard_parts:polyfuse_5.1mm" H 7850 6100 50  0001 L CNN
 F 3 "~" H 7800 6300 50  0001 C CNN

Commit message: Update discipline-pcb.sch
Parts:
- added SW69: KEYSW, cftkb:SW_Cherry_MX1A_1.25u_PCBNOSCREEN, symbol keyboard_parts:KEYSW
- added SW70, SW71, SW73, SW74: KEYSW, cftkb:SW_Cherry_MX1A_1.50u_PCBNOSCREEN, symbol keyboard_parts:KEYSW
- added SW72: KEYSW, Button_Switch_Keyboard:SW_Cherry_MX1A_1.00u_PCB-NOSCREEN, symbol keyboard_parts:KEYSW
- BOOT1, RESET1: footprint Button_Switch_THT:SW_PUSH_6mm -> cftkb:SW_PUSH_6mm
- C1, C2: footprint Capacitor_THT:C_Disc_D3.0mm_W1.6mm_P2.50mm -> cftkb:C_Disc_D3.0mm_W1.6mm_P2.50mm
- C3: footprint Capacitor_THT:CP_Radial_D4.0mm_P1.50mm -> cftkb:CP_Radial_D4.0mm_P1.50mm
- C4, C5: footprint Capacitor_THT:C_Disc_D4.3mm_W1.9mm_P5.00mm -> cftkb:C_Disc_D4.3mm_W1.9mm_P5.00mm
- D1, D10, D11, D12, D13, D14, D15, D16, D17, D18, D19, D2, D20, D21, D22, D23, D24, D25, D26, D27, D28, D29, D3, D30, D31, D32, D33, D34, D35, D36, D37, D38, D39, D4, D40, D41, D42, D43, D44, D45, D46, D47, D48, D49, D5, D50, D51, D52, D53, D54, D55, D56, D57, D58, D59, D6, D60, D61, D62, D63, D64, D65, D66, D67, D68, D69, D7, D70, D8, D9: footprint Diode_THT:D_DO-35_SOD27_P5.08mm_Horizontal -> cftkb:D_DO-35_SOD27_P5.08mm_Horizontal
- F1: footprint keyboard_parts:polyfuse_5.1mm -> cftkb:polyfuse_5.1mm
- J1: footprint (none) -> cftkb:AVR_ICSP_3x2
- R1, R2, R3, R4, R5, R6, R7: footprint Resistor_THT:R_Axial_DIN0204_L3.6mm_D1.6mm_P7.62mm_Horizontal -> cftkb:R_Axial_DIN0204_L3.6mm_D1.6mm_P7.62mm_Horizontal
- SW1, SW10, SW11, SW12, SW13, SW15, SW17, SW18, SW19, SW2, SW20, SW21, SW22, SW23, SW24, SW25, SW26, SW27, SW28, SW3, SW30, SW32, SW33, SW34, SW35, SW36, SW37, SW38, SW39, SW4, SW40, SW41, SW42, SW44, SW46, SW47, SW48, SW49, SW5, SW50, SW51, SW52, SW53, SW54, SW55, SW57, SW58, SW6, SW62, SW65, SW66, SW67, SW68, SW7, SW8, SW9: footprint Button_Switch_Keyboard:SW_Cherry_MX1A_1.00u_PCB-NOSCREEN -> cftkb:SW_Cherry_MX1A_1.00u_PCB-NOSCREEN
- SW14: footprint Button_Switch_Keyboard:SW_Cherry_MX1A_2.00u_PCBNOSCREEN -> cftkb:SW_Cherry_MX1A_2.00u_PCBNOSCREEN
- SW16, SW29: footprint Button_Switch_Keyboard:SW_Cherry_MX1A_1.50u_PCBNOSCREEN -> cftkb:SW_Cherry_MX1A_1.50u_PCBNOSCREEN
- SW31, SW56: footprint Button_Switch_Keyboard:SW_Cherry_MX1A_1.75u_PCBNOSCREEN -> cftkb:SW_Cherry_MX1A_1.75u_PCBNOSCREEN
- SW43, SW45: footprint Button_Switch_Keyboard:SW_Cherry_MX1A_2.25u_PCBNOSCREEN -> cftkb:SW_Cherry_MX1A_2.25u_PCBNOSCREEN
- SW59, SW60, SW61, SW63, SW64: footprint Button_Switch_Keyboard:SW_Cherry_MX1A_1.25u_PCBNOSCREEN -> cftkb:SW_Cherry_MX1A_1.25u_PCBNOSCREEN
- USB1: footprint Type-C:USB_C_GCT_USB4085 -> cftkb:USB_C_GCT_USB4085
- Y1: footprint Crystal:Crystal_HC49-4H_Vertical -> cftkb:Crystal_HC49-4H_Vertical
Connections:
- wire segments 271 -> 339

Commit message: Revert "Update discipline-pcb.sch"
This reverts commit a72fcd6089ef7a7854f28251b3b3dd299a3c70af.
Parts:
- removed SW69: KEYSW, cftkb:SW_Cherry_MX1A_1.25u_PCBNOSCREEN, symbol keyboard_parts:KEYSW
- removed SW70, SW71, SW73, SW74: KEYSW, cftkb:SW_Cherry_MX1A_1.50u_PCBNOSCREEN, symbol keyboard_parts:KEYSW
- removed SW72: KEYSW, Button_Switch_Keyboard:SW_Cherry_MX1A_1.00u_PCB-NOSCREEN, symbol keyboard_parts:KEYSW
- BOOT1, RESET1: footprint cftkb:SW_PUSH_6mm -> Button_Switch_THT:SW_PUSH_6mm
- C1, C2: footprint cftkb:C_Disc_D3.0mm_W1.6mm_P2.50mm -> Capacitor_THT:C_Disc_D3.0mm_W1.6mm_P2.50mm
- C3: footprint cftkb:CP_Radial_D4.0mm_P1.50mm -> Capacitor_THT:CP_Radial_D4.0mm_P1.50mm
- C4, C5: footprint cftkb:C_Disc_D4.3mm_W1.9mm_P5.00mm -> Capacitor_THT:C_Disc_D4.3mm_W1.9mm_P5.00mm
- D1, D10, D11, D12, D13, D14, D15, D16, D17, D18, D19, D2, D20, D21, D22, D23, D24, D25, D26, D27, D28, D29, D3, D30, D31, D32, D33, D34, D35, D36, D37, D38, D39, D4, D40, D41, D42, D43, D44, D45, D46, D47, D48, D49, D5, D50, D51, D52, D53, D54, D55, D56, D57, D58, D59, D6, D60, D61, D62, D63, D64, D65, D66, D67, D68, D69, D7, D70, D8, D9: footprint cftkb:D_DO-35_SOD27_P5.08mm_Horizontal -> Diode_THT:D_DO-35_SOD27_P5.08mm_Horizontal
- F1: footprint cftkb:polyfuse_5.1mm -> keyboard_parts:polyfuse_5.1mm
- J1: footprint cftkb:AVR_ICSP_3x2 -> (none)
- R1, R2, R3, R4, R5, R6, R7: footprint cftkb:R_Axial_DIN0204_L3.6mm_D1.6mm_P7.62mm_Horizontal -> Resistor_THT:R_Axial_DIN0204_L3.6mm_D1.6mm_P7.62mm_Horizontal
- SW1, SW10, SW11, SW12, SW13, SW15, SW17, SW18, SW19, SW2, SW20, SW21, SW22, SW23, SW24, SW25, SW26, SW27, SW28, SW3, SW30, SW32, SW33, SW34, SW35, SW36, SW37, SW38, SW39, SW4, SW40, SW41, SW42, SW44, SW46, SW47, SW48, SW49, SW5, SW50, SW51, SW52, SW53, SW54, SW55, SW57, SW58, SW6, SW62, SW65, SW66, SW67, SW68, SW7, SW8, SW9: footprint cftkb:SW_Cherry_MX1A_1.00u_PCB-NOSCREEN -> Button_Switch_Keyboard:SW_Cherry_MX1A_1.00u_PCB-NOSCREEN
- SW14: footprint cftkb:SW_Cherry_MX1A_2.00u_PCBNOSCREEN -> Button_Switch_Keyboard:SW_Cherry_MX1A_2.00u_PCBNOSCREEN
- SW16, SW29: footprint cftkb:SW_Cherry_MX1A_1.50u_PCBNOSCREEN -> Button_Switch_Keyboard:SW_Cherry_MX1A_1.50u_PCBNOSCREEN
- SW31, SW56: footprint cftkb:SW_Cherry_MX1A_1.75u_PCBNOSCREEN -> Button_Switch_Keyboard:SW_Cherry_MX1A_1.75u_PCBNOSCREEN
- SW43, SW45: footprint cftkb:SW_Cherry_MX1A_2.25u_PCBNOSCREEN -> Button_Switch_Keyboard:SW_Cherry_MX1A_2.25u_PCBNOSCREEN
- SW59, SW60, SW61, SW63, SW64: footprint cftkb:SW_Cherry_MX1A_1.25u_PCBNOSCREEN -> Button_Switch_Keyboard:SW_Cherry_MX1A_1.25u_PCBNOSCREEN
- USB1: footprint cftkb:USB_C_GCT_USB4085 -> Type-C:USB_C_GCT_USB4085
- Y1: footprint cftkb:Crystal_HC49-4H_Vertical -> Crystal:Crystal_HC49-4H_Vertical
Connections:
- wire segments 339 -> 271

Commit message: Change to Mini USB port
Parts:
- removed R1, R2: 5.1k, Resistor_THT:R_Axial_DIN0204_L3.6mm_D1.6mm_P7.62mm_Horizontal, symbol Device:R_Small
- removed USB1: USB_C_GCT_USB4085, Type-C:USB_C_GCT_USB4085, symbol Type-C:USB_C_GCT_USB4085
- added J-USB-1: USB_B_Mini, Projects:USB_MINIB_Akizuki_MUSB-5BF01AS, symbol Connector:USB_B_Mini
- BOOT1, RESET1: symbol keyboard_parts:SW_PUSH -> discipline-pcb-rescue:SW_PUSH-keyboard_parts
- J1: symbol Connector:AVR-ISP-6 -> discipline-pcb-rescue:AVR-ISP-6-Connector
- SW1, SW10, SW11, SW12, SW13, SW14, SW15, SW16, SW17, SW18, SW19, SW2, SW20, SW21, SW22, SW23, SW24, SW25, SW26, SW27, SW28, SW29, SW3, SW30, SW31, SW32, SW33, SW34, SW35, SW36, SW37, SW38, SW39, SW4, SW40, SW41, SW42, SW43, SW44, SW45, SW46, SW47, SW48, SW49, SW5, SW50, SW51, SW52, SW53, SW54, SW55, SW56, SW57, SW58, SW59, SW6, SW60, SW61, SW62, SW63, SW64, SW65, SW66, SW67, SW68, SW7, SW8, SW9: symbol keyboard_parts:KEYSW -> discipline-pcb-rescue:KEYSW-keyboard_parts
- U1: symbol MCU_Microchip_ATmega:ATmega32A-PU -> discipline-pcb-rescue:ATmega32A-PU-MCU_Microchip_ATmega
Connections:
- wire segments 271 -> 312
- no-connect marks 9 -> 8
Other:
- moved on the sheet: J1
