File: discipline-pcb.sch (KiCad schematic (older format))
At the start: 164 parts, among them J1 AVR-ISP-6, SW1 KEYSW, SW10 KEYSW, SW11 KEYSW, SW12 KEYSW, SW13 KEYSW, SW14 KEYSW, SW15 KEYSW, SW16 KEYSW, SW17 KEYSW, SW18 KEYSW, SW19 KEYSW, SW2 KEYSW, SW20 KEYSW, SW21 KEYSW, SW22 KEYSW, SW23 KEYSW, SW24 KEYSW, SW25 KEYSW, SW26 KEYSW, SW27 KEYSW, SW28 KEYSW, SW29 KEYSW, SW3 KEYSW, SW30 KEYSW, SW31 KEYSW, SW32 KEYSW, SW33 KEYSW, SW34 KEYSW, SW35 KEYSW, SW36 KEYSW, SW37 KEYSW, SW38 KEYSW, SW39 KEYSW, SW4 KEYSW, SW40 KEYSW, SW41 KEYSW, SW42 KEYSW, SW43 KEYSW, SW44 KEYSW, SW45 KEYSW, SW46 KEYSW, SW47 KEYSW, SW48 KEYSW, SW49 KEYSW, SW5 KEYSW, SW50 KEYSW, SW51 KEYSW, SW52 KEYSW, SW53 KEYSW, SW54 KEYSW, SW55 KEYSW, SW56 KEYSW, SW57 KEYSW, SW58 KEYSW, SW59 KEYSW, SW6 KEYSW, SW60 KEYSW, SW61 KEYSW, SW62 KEYSW, SW63 KEYSW, SW64 KEYSW, SW65 KEYSW, SW66 KEYSW, SW67 KEYSW, SW68 KEYSW, SW69 KEYSW, SW7 KEYSW, SW70 KEYSW, SW71 KEYSW, SW72 KEYSW, SW73 KEYSW, SW74 KEYSW, SW8 KEYSW, SW9 KEYSW, U1 ATmega32A-PU, Y1 Crystal

Commit message: Update discipline-pcb.sch
Parts:
- removed U1: ATmega32A-PU, cftkb:DIP-40_W15.24mm, symbol discipline-pcb-rescue:ATmega32A-PU-MCU_Microchip_ATmega
- added U1: ATmega32A-PU, cftkb:DIP-40_W15.24mm, symbol MCU_Microchip_ATmega:ATmega32A-PU
Connections:
- net +5V: now also U1.10 (VCC), U1.30 (AVCC)
- net D+: now also U1.16 (PD2)
- net D-: now also U1.17 (PD3)
- net GND: now also U1.11 (GND), U1.31 (GND)
- net MISO: now also U1.7 (PB6)
- net MOSI: now also U1.6 (PB5)
- net SCK: now also U1.8 (PB7)
- net boot: now also U1.18 (PD4)
- net col0: now also U1.38 (PA2)
- net col1: now also U1.4 (PB3)
- net col10: now also U1.25 (PC3)
- net col11: now also U1.24 (PC2)
- net col12: now also U1.23 (PC1)
- net col13: now also U1.22 (PC0)
- net col14: now also U1.21 (PD7)
- net col2: now also U1.37 (PA3)
- net col3: now also U1.5 (PB4)
- net col4: now also U1.36 (PA4)
- net col5: now also U1.19 (PD5)
- net col6: now also U1.20 (PD6)
- net col7: now also U1.28 (PC6)
- net col8: now also U1.27 (PC5)
- net col9: now also U1.26 (PC4)
- net reset: now also U1.9 (~RESET)
- net row0: now also U1.3 (PB2)
- net row1: now also U1.39 (PA1)
- net row2: now also U1.2 (PB1)
- net row3: now also U1.40 (PA0)
- net row4: now also U1.1 (PB0)
- net at C2.1, Y1.2: now also U1.12 (XTAL2)
- net at C1.1, Y1.1: now also U1.13 (XTAL1)
Changed lines of the file:
@@
 Text GLabel 5800 6900 2    50   Input ~ 0
 reset
-$Comp
-L discipline-pcb-rescue:ATmega32A-PU-MCU_Microchip_ATmega U1
-U 1 1 5D1828C7
-P 4000 8250
-F 0 "U1" H 3800 8400 50  0000 C CNN
-F 1 "ATmega32A-PU" H 3850 8300 50  0000 C CNN
-F 2 "cftkb:DIP-40_W15.24mm" H 4000 8250 50  0001 C CIN
-F 3 "http://ww1.microchip.com/downloads/en/DeviceDoc/atmel-8155-8-bit-microcontroller-avr-atmega32a_datasheet.pdf" H 4000 8250 50  0001 C CNN
-	1    4000 8250
-	1    0    0    -1
-$EndComp
 Wire Wire Line
 	4000 6250 4100 6250
@@
 	10550 5900 10550 5250
 Connection ~ 10550 5250
+$Comp
+L MCU_Microchip_ATmega:ATmega32A-PU U1
+U 1 1 5DF0B623
+P 4000 8250
+F 0 "U1" H 3850 8350 50  0000 C CNN
+F 1 "ATmega32A-PU" H 3900 8250 50  0000 C CNN
+F 2 "cftkb:DIP-40_W15.24mm" H 4000 8250 50  0001 C CIN
+F 3 "http://ww1.microchip.com/downloads/en/DeviceDoc/atmel-8155-8-bit-microcontroller-avr-atmega32a_datasheet.pdf" H 4000 8250 50  0001 C CNN
+	1    4000 8250
+	1    0    0    -1
+$EndComp
+Connection ~ 4100 6250
 $EndSCHEMATC

Commit message: Update to V2, add ISO support, update license
Parts:
- added D71: (no value), cftkb:D_DO-35_SOD27_P5.08mm_Horizontal, symbol Device:D
- added SW75, SW77: KEYSW, cftkb:SW_Cherry_MX1A_1.00u_PCB-NOSCREEN, symbol keyboard_parts:KEYSW
- added SW76: KEYSW, cftkb:SW_Cherry_MX1A_ISOEnter_PCB_ReversedStabilizer, symbol keyboard_parts:KEYSW
- added SW78: KEYSW, cftkb:SW_Cherry_MX1A_1.25u_PCBNOSCREEN, symbol keyboard_parts:KEYSW
- C1, C2: footprint cftkb:D_DO-35_SOD27_P5.08mm_Horizontal -> cftkb:C_Disc_D3.0mm_W1.6mm_P2.50mm
- C3: footprint cftkb:D_DO-35_SOD27_P5.08mm_Horizontal -> cftkb:CP_Radial_D4.0mm_P1.50mm
- C4, C5: footprint cftkb:D_DO-35_SOD27_P5.08mm_Horizontal -> cftkb:C_Disc_D4.3mm_W1.9mm_P5.00mm
- J1: symbol Connector:AVR-ISP-6 -> discipline-pcb-rescue:AVR-ISP-6-Connector
- R1, R2, R3, R4, R5, R6, R7: footprint cftkb:R_Axial_DIN0204_L3.6mm_D1.6mm_P7.62mm_Horizontal -> cftkb:R_Axial_DIN0204_L3.6mm_D1.6mm_P5.08mm_Horizontal
- U1: symbol MCU_Microchip_ATmega:ATmega32A-PU -> discipline-pcb-rescue:ATmega32A-PU-MCU_Microchip_ATmega
Connections:
- net GND: now also BOOT1.2, RESET1.2; no longer BOOT1.1, RESET1.1
- net boot: now also BOOT1.1; no longer BOOT1.2
- net col0: now also SW78.1
- net col1: now also SW75.1
- net col13: now also SW76.1, SW77.1
- net reset: now also RESET1.1; no longer RESET1.2
- net row3: now also D71.1 (K)
- net at D29.2 (A), SW29.2: now also SW76.2
- net at D43.2 (A), SW43.2: now also SW77.2
- net at D45.2 (A), SW45.2: now also SW78.2
- new net: D71.2 (A), SW75.2
Other:
- note added: "1.1"
- note added: "1/1/2020"
- note added: "ISP"
- note added: "MCU"
- note added: "POWER"
- note added: "POWER LED"
- note added: "RESET"
- note added: "USB"
- note removed: "1"
- note removed: "7/1/2019"
- moved on the sheet: BOOT1, C1, C2, C3, C4, C5, D69, D70, F1, J1, LED1, R1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

Commit message: Update discipline-pcb.sch
Parts:
- removed Y1: Crystal, cftkb:Crystal_HC49-4H_Vertical, symbol Device:Crystal
- added Y1: Crystal, cftkb:Crystal_HC49-4H_Vertical, symbol Device:Crystal_Small
Connections:
- net at C1.1, U1.13 (XTAL1): now also Y1.1
- net at C2.1, U1.12 (XTAL2): now also Y1.2
Changed lines of the file:
@@
 D+
-$Comp
-L Device:Crystal Y1
-U 1 1 5D1F9BED
-P 2975 7300
-F 0 "Y1" V 2929 7431 50  0000 L CNN
-F 1 "Crystal" V 3020 7431 50  0000 L CNN
-F 2 "cftkb:Crystal_HC49-4H_Vertical" H 2975 7300 50  0001 C CNN
-F 3 "~" H 2975 7300 50  0001 C CNN
-	1    2975 7300
-	0    1    1    0
-$EndComp
-Wire Wire Line
-	2975 7150 3225 7150
-Wire Wire Line
-	3225 7150 3225 7200
-Wire Wire Line
-	3225 7200 3375 7200
-Wire Wire Line
-	2975 7450 3225 7450
-Wire Wire Line
-	3225 7450 3225 7400
-Wire Wire Line
-	3225 7400 3375 7400
 $Comp
 L Device:C_Small C2
@@
 	1    0    0    -1
 $EndComp
-Wire Wire Line
-	2975 7450 2975 7550
-Connection ~ 2975 7450
-Wire Wire Line
-	2975 7150 2825 7150
-Wire Wire Line
-	2825 7150 2825 7550
-Connection ~ 2975 7150
 Wire Wire Line
 	2825 7750 2975 7750
@@
 	1    0    0    -1
 $EndComp
+$Comp
+L Device:Crystal_Small Y1
+U 1 1 5F0E7676
+P 2975 7300
+F 0 "Y1" V 2929 7388 50  0000 L CNN
+F 1 "Crystal" V 3020 7388 50  0000 L CNN
+F 2 "cftkb:Crystal_HC49-4H_Vertical" H 2975 7300 50  0001 C CNN
+F 3 "~" H 2975 7300 50  0001 C CNN
+	1    2975 7300
+	0    1    1    0
+$EndComp
+Wire Wire Line
+	3375 7200 2975 7200
+Wire Wire Line
+	3375 7400 2975 7400
+Wire Wire Line
+	2975 7400 2975 7550
+Connection ~ 2975 7400
+Wire Wire Line
+	2975 7200 2825 7200
+Wire Wire Line
+	2825 7200 2825 7550
+Connection ~ 2975 7200
 $EndSCHEMATC

Commit message: Add missing keyboard_parts.lib, fix symbol refs in schematic
Parts:
- J1: symbol discipline-pcb-rescue:AVR-ISP-6-Connector -> Connector:AVR-ISP-6
- U1: symbol discipline-pcb-rescue:ATmega32A-PU-MCU_Microchip_ATmega -> MCU_Microchip_ATmega:ATmega32A-PU
- USB1: symbol Type-C:USB_C_GCT_USB4085 -> Connector:USB_C_Receptacle_USB2.0
Other:
- moved on the sheet: D69, D70, F1, J1, R1, R2, R3, R4, R5
