File: bottom/discipline-pcb.kicad_pcb (KiCad board)
At the start: 2 copper layers, 304.9 x 122.8 mm, 15 parts

Commit message: update screenprint and gerbers
Other:
- board text removed: "JLCJLCJLCJLC"
Changed lines of the file:
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@@
   (general
     (thickness 1.6)
-    (drawings 14)
+    (drawings 13)
     (tracks 0)
     (zones 0)
@@
     (pad 1 thru_hole circle (at 0 0) (size 8.6 8.6) (drill 4.3) (layers *.Cu *.Mask))
   )
-  (gr_text JLCJLCJLCJLC (at 307.923938 67.243533) (layer F.SilkS)
-    (effects (font (size 0.9 0.9) (thickness 0.16)))
-  )
   (gr_text coseyfannitutti (at 118.1115 133.50974) (layer B.Mask)

Commit message: Update to V2, add ISO support, update license
Parts:
- removed the G*** at (128.2, 133.8) (x2)
- removed the REF** at (337.2, 91.4)
- removed the REF** at (88.7, 91.4)
- added G***: LOGO, logos:coseyfannitutti_rev1_16mm_copper, F.Cu at (300.8, 132.5)
- added G***: LOGO, logos:coseyfannitutti_16mm, F.Cu at (300.8, 132.5)
- added G***: LOGO, logos:TOPY 3MM MASK, F.Cu at (291.2, 133.9)
- added G***: LOGO, logos:TOPY 3MM COPPER, F.Cu at (291.2, 133.9)
- added REF**: MountingHole_2.2mm_M2_Pad, MountingHole:MountingHole_2.2mm_M2_Pad, F.Cu at (206.2, 92.4)
- added REF**: MountingHole_2.2mm_M2_Pad, MountingHole:MountingHole_2.2mm_M2_Pad, F.Cu at (82.0, 92.4)
- added REF**: MountingHole_2.2mm_M2_Pad, MountingHole:MountingHole_2.2mm_M2_Pad, F.Cu at (330.5, 92.4)
- added REF**: MountingHole_2.2mm_M2_Pad, MountingHole:MountingHole_2.2mm_M2_Pad, F.Cu at (206.2, 61.7)
- added REF**: MountingHole_2.2mm_M2_Pad, MountingHole:MountingHole_2.2mm_M2_Pad, F.Cu at (206.2, 80.4)
- G***: moved to F.Cu
- moved REF** 8.97 mm to (57.8, 80.4)
- moved REF** 8.74 mm to (57.8, 61.7)
- moved REF** 8.28 mm to (315.9, 161.1)
- moved REF** 8.28 mm to (298.7, 104.3)
- moved H1 8.28 mm to (206.2, 167.0)
- moved REF** 8.28 mm to (96.6, 161.1)
- moved REF** 8.28 mm to (206.2, 104.3)
- moved REF** 8.28 mm to (113.8, 104.3)
- moved REF** 7.86 mm to (354.7, 80.4)
- moved REF** 7.60 mm to (354.7, 61.7)
- moved G*** 6.12 mm to (209.8, 118.8), turned to 0 degrees
Routing:
- net GND: vias 0 -> 1
Other:
- board text added: "1.1"
- board text added: "7/2/2019 - updated 12/3/2019"
- board text added: "DISCIPLINE - 65% keyboard assembled with only through hole components"
- board text removed: "1"
- board text removed: "7/2/2019"
- board text removed: "DISCIPLINE - 65% keyboard made with only through hole components"
- board text removed: "coseyfannitutti"
